Commit message: update path needed for gz

File: tiago_pro_description/ros2_control/ros2_control.urdf.xacro (robot description, xacro)
@@ -143,5 +143,5 @@
       <!-- Init the ROS 2 control gazebo interface -->
       <gazebo>
-        <plugin filename="libgazebo_ros2_control.so" name="gazebo_ros2_control">
+        <plugin filename="libgz_ros2_control-system.so" name="gz_ros2_control::GazeboSimROS2ControlPlugin">
           <parameters>$(find tiago_pro_description)/ros2_control/gazebo_controller_manager_cfg.yaml</parameters>
         </plugin>
@@ -149,5 +149,5 @@
       <ros2_control name="ros2_control_gazebo_system" type="system">
         <hardware>
-          <plugin>gazebo_ros2_control/GazeboSystem</plugin>
+          <plugin>gz_ros2_control/GazeboSimSystem</plugin>
         </hardware>
         <!-- wheels -->

File: tiago_pro_description/urdf/pilot_station/basestation.urdf.xacro (robot description, xacro)
@@ -36,5 +36,5 @@
           rpy="0 0 0" />
         <geometry>
-            <mesh filename="package://tiago_pro_description/meshes/pilot_station/fixed_sit_station.stl" />
+            <mesh filename="file://$(find tiago_pro_description)/meshes/pilot_station/fixed_sit_station.stl" />
         </geometry>
         <material
@@ -49,5 +49,5 @@
           rpy="0 0 0" />
         <geometry>
-            <mesh filename="package://tiago_pro_description/meshes/pilot_station/fixed_sit_station.stl" />
+            <mesh filename="file://$(find tiago_pro_description)/meshes/pilot_station/fixed_sit_station.stl" />
         </geometry>
       </collision>

File: tiago_pro_description/urdf/pilot_station/teleop_handle.urdf.xacro (robot description, xacro)
@@ -36,5 +36,5 @@
         rpy="0 0 0" />
       <geometry>
-          <mesh filename="package://tiago_pro_description/meshes/pilot_station/teleop_handle.stl" />
+          <mesh filename="file://$(find tiago_pro_description)/meshes/pilot_station/teleop_handle.stl" />
       </geometry>
       <material
@@ -49,5 +49,5 @@
         rpy="0 0 0" />
       <geometry>
-          <mesh filename="package://tiago_pro_description/meshes/pilot_station/teleop_handle.stl" />
+          <mesh filename="file://$(find tiago_pro_description)/meshes/pilot_station/teleop_handle.stl" />
       </geometry>
     </collision>

File: tiago_pro_description/urdf/torso/torso.urdf.xacro (robot description, xacro)
@@ -27,5 +27,5 @@
         <origin xyz="0 0 0" rpy="0 0 0" />
         <geometry>
-          <mesh filename="package://tiago_pro_description/meshes/torso/torso_fixed.stl" />
+          <mesh filename="file://$(find tiago_pro_description)/meshes/torso/torso_fixed.stl" />
         </geometry>
         <material name="pal/DarkGrey"/>
@@ -34,5 +34,5 @@
         <origin xyz="0 0 0" rpy="0 0 0" />
         <geometry>
-          <mesh filename="package://tiago_pro_description/meshes/torso/torso_fixed_collision.stl" />
+          <mesh filename="file://$(find tiago_pro_description)/meshes/torso/torso_fixed_collision.stl" />
         </geometry>
       </collision>
@@ -76,5 +76,5 @@
         <origin xyz="0 0 0" rpy="0 0 0" />
         <geometry>
-          <mesh filename="package://tiago_pro_description/meshes/torso/torso_lift_link.stl" />
+          <mesh filename="file://$(find tiago_pro_description)/meshes/torso/torso_lift_link.stl" />
         </geometry>
         <material name="">
@@ -85,5 +85,5 @@
         <origin xyz="0 0 0" rpy="0 0 0" />
         <geometry>
-          <mesh filename="package://tiago_pro_description/meshes/torso/torso_lift_link_collision.stl" />
+          <mesh filename="file://$(find tiago_pro_description)/meshes/torso/torso_lift_link_collision.stl" />
         </geometry>
       </collision>
@@ -91,5 +91,5 @@
         <origin xyz="-0.226436438571948 3.12797385809451E-05 0.00524038105676683" rpy="0 0 -1.5707963267949" />
         <geometry>
-          <mesh filename="package://tiago_pro_description/meshes/torso/laptop_tray_collision.stl" />
+          <mesh filename="file://$(find tiago_pro_description)/meshes/torso/laptop_tray_collision.stl" />
         </geometry>
       </collision>

Commit message: try to fix gripper mimic (not working yet)

File: tiago_pro_description/ros2_control/ros2_control.urdf.xacro (robot description, xacro)
@@ -29,5 +29,5 @@
     </ros2_control>
   </xacro:macro>
-  <xacro:macro name="ros2_control_arms">
+  <xacro:macro name="ros2_control_arms" params="sim_type:=no-simulation">
     <!-- arm left -->
     <xacro:if value="${has_arm_left}">
@@ -44,5 +44,5 @@
       </xacro:if>
       <xacro:if value="${end_effector_left == 'pal-pro-gripper'}">
-        <xacro:ros2_control_pal_pro_gripper name="gripper_left" reduction="1.0" />
+        <xacro:ros2_control_pal_pro_gripper name="gripper_left" reduction="1.0" sim_type="${sim_type}"/>
       </xacro:if>
     </xacro:if>
@@ -62,5 +62,5 @@
       <xacro:if value="${end_effector_right == 'pal-pro-gripper'}">
         <!-- pal-pro-gripper -->
-        <xacro:ros2_control_pal_pro_gripper name="gripper_right" reduction="1.0" />
+        <xacro:ros2_control_pal_pro_gripper name="gripper_right" reduction="1.0" sim_type="${sim_type}"/>
       </xacro:if>
     </xacro:if>
@@ -158,5 +158,5 @@
         <xacro:ros2_control_head_offset />
         <!-- arms -->
-        <xacro:ros2_control_arms/>
+        <xacro:ros2_control_arms sim_type="gazebo"/>
         <xacro:arg name="pid_controllers" default="false"/>
         <xacro:if value="${end_effector_right == 'allegro-hand'}">
