Commit message: Wire sim_type to the gripper and enable the gripper_grasper wrapper
Companion to the pal_pro_gripper mimic joint fix. Threads sim_type down to the gripper's ros2_control config, lowers position_proportional_gain to reduce overshoot into joint limits, and enables the gripper_grasper launch (was commented out) so /grasp and /release come up by default.

File: tiago_pro_description/ros2_control/ros2_control.urdf.xacro (robot description, xacro)
@@ -29,5 +29,5 @@
     </ros2_control>
   </xacro:macro>
-  <xacro:macro name="ros2_control_arms">
+  <xacro:macro name="ros2_control_arms" params="sim_type:=no-simulation">
     <!-- arm left -->
     <xacro:if value="${has_arm_left}">
@@ -44,5 +44,5 @@
       </xacro:if>
       <xacro:if value="${end_effector_left == 'pal-pro-gripper'}">
-        <xacro:ros2_control_pal_pro_gripper name="gripper_left" reduction="1.0" />
+        <xacro:ros2_control_pal_pro_gripper name="gripper_left" reduction="1.0" sim_type="${sim_type}" />
       </xacro:if>
     </xacro:if>
@@ -62,5 +62,5 @@
       <xacro:if value="${end_effector_right == 'pal-pro-gripper'}">
         <!-- pal-pro-gripper -->
-        <xacro:ros2_control_pal_pro_gripper name="gripper_right" reduction="1.0" />
+        <xacro:ros2_control_pal_pro_gripper name="gripper_right" reduction="1.0" sim_type="${sim_type}" />
       </xacro:if>
     </xacro:if>
@@ -89,8 +89,8 @@
         </xacro:if>
         <xacro:if value="${end_effector_teleop_right == 'pal-pro-gripper'}">
-          <xacro:ros2_control_pal_pro_gripper name="gripper_teleop_right" reduction="1.0" />
+          <xacro:ros2_control_pal_pro_gripper name="gripper_teleop_right" reduction="1.0" sim_type="${sim_type}" />
         </xacro:if>
         <xacro:if value="${end_effector_teleop_left == 'pal-pro-gripper'}">
-          <xacro:ros2_control_pal_pro_gripper name="gripper_teleop_left" reduction="1.0" />
+          <xacro:ros2_control_pal_pro_gripper name="gripper_teleop_left" reduction="1.0" sim_type="${sim_type}" />
         </xacro:if>
     </xacro:if>
@@ -158,5 +158,5 @@
         <xacro:ros2_control_head_offset />
         <!-- arms -->
-        <xacro:ros2_control_arms/>
+        <xacro:ros2_control_arms sim_type="gazebo"/>
         <xacro:arg name="pid_controllers" default="false"/>
         <xacro:if value="${end_effector_right == 'allegro-hand'}">
@@ -213,5 +213,5 @@
         </hardware>
         <!-- arms -->
-        <xacro:ros2_control_arms/>
+        <xacro:ros2_control_arms sim_type="no-simulation"/>
         <xacro:ros2_control_torso name="torso_lift" reduction="1.0" />
       </ros2_control>
